Commit message: Physical model not explode

File: bme_ros_simple_arm/urdf/tomi_arm.xacro (robot description, xacro)
@@ -16,9 +16,9 @@
   <link name="link_0">
     <inertial>
-      <mass value="2"/>
-      <origin xyz="0.0 0.0 0.0"/>
-      <inertia ixx="0.0117" ixy="0.0" ixz="0.0"
-               iyy="0.0117" iyz="0.0"
-               izz="0.0225"
+      <mass value="7.57"/>
+      <origin xyz="0.0 0.0 0.0957"/>
+      <inertia ixx="0.0368" ixy="0.0" ixz="0.0"
+               iyy="0.0368" iyz="0.0"
+               izz="0.0273"
       />
     </inertial>
@@ -31,5 +31,5 @@
     <visual>
       <geometry>
-        <mesh scale = "0.001 0.001 0.001" filename = "package://bme_ros_simple_arm/meshes/link0.dae"/>
+        <mesh scale = "1 1 1" filename = "package://bme_ros_simple_arm/meshes/Link0.dae"/>
       </geometry>
       <material name="grey"/>
@@ -42,5 +42,5 @@
   <!-- Axis1 - Link 0 - Link 1 -->
   <joint name="Axis1" type="revolute">
-    <limit lower="-2.6179" upper="2.6179" effort="0" velocity="7.33"/> <!-- +-150° , 420°/s which is 7.33 rad/s-->
+    <limit lower="-2.6179" upper="2.6179" effort="5" velocity="7.33"/> <!-- +-150° , 420°/s which is 7.33 rad/s-->
     <parent link="link_0"/>
     <child link="link_1"/>
@@ -53,9 +53,9 @@
   <link name="link_1">
     <inertial>
-      <mass value="0.5"/>
-      <origin xyz="0.0 0.0 0.0" rpy="0.0 0.0 0.0"/>
-      <inertia ixx="0.0014" ixy="0.0" ixz="0.0"
-               iyy="0.0014" iyz="0.0"
-               izz="0.0025"
+      <mass value="6.09"/>
+      <origin xyz="0.142 0.0 0.043" rpy="0.0 0.0 0.0"/>
+      <inertia ixx="0.0174" ixy="0.0" ixz="0.0"
+               iyy="0.1039" iyz="0.0"
+               izz="0.1138"
       />
     </inertial>
@@ -68,5 +68,5 @@
     <visual>
       <geometry>
-        <mesh scale = "0.001 0.001 0.001" filename = "package://bme_ros_simple_arm/meshes/link1.dae"/>
+        <mesh scale = "1 1 1" filename = "package://bme_ros_simple_arm/meshes/Link1.dae"/>
       </geometry>
       <material name="orange"/>
@@ -79,10 +79,10 @@
   <!-- Joint 2 - Link 1 - Link 2 -->
   <joint name="Axis2" type="revolute">
-    <limit lower="-2.5307" upper="2.5307" effort="0" velocity="12.23"/> <!-- +- 145° which is +- 2.5307 rad , 701°/s which is 12.23 rad/s -->
+    <limit lower="-2.5307" upper="2.5307" effort="5" velocity="12.23"/> <!-- +- 145° which is +- 2.5307 rad , 701°/s which is 12.23 rad/s -->
     <parent link="link_1"/>
     <child link="link_2"/>
     <axis xyz="0 0 1"/>
-    <origin xyz="0.290 0.0 0.09" rpy="0.0 0.0 0.0"/>
-    <!--<origin xyz="0.290 0.0 0.086" rpy="0.0 0.0 0.0"/>-->
+    <!--<origin xyz="0.290 0.0 0.09" rpy="0.0 0.0 0.0"/>-->
+    <origin xyz="0.290 0.0 0.086" rpy="0.0 0.0 0.0"/>
     <dynamics damping="0.0" friction="0.0"/>
   </joint>
@@ -90,9 +90,9 @@
   <link name="link_2">
     <inertial>
-      <mass value="0.3"/>
-      <origin xyz="0.0 0.0 0.0" rpy="0.0 0.0 0.0"/>
-      <inertia ixx="0.0012" ixy="0.0" ixz="0.0"
-               iyy="0.0012" iyz="0.0"
-               izz="0.0004"
+      <mass value="9.01"/>
+      <origin xyz="0.1075 0.0 0.089" rpy="0.0 0.0 0.0"/>
+      <inertia ixx="0.0398" ixy="0.0" ixz="0.0"
+               iyy="0.1764" iyz="0.0"
+               izz="0.1686"
       />
     </inertial>
@@ -105,5 +105,5 @@
     <visual>
       <geometry>
-        <mesh scale = "0.001 0.001 0.001" filename = "package://bme_ros_simple_arm/meshes/link2.dae"/>
+        <mesh scale = "1 1 1" filename = "package://bme_ros_simple_arm/meshes/Link2.dae"/>
         <!--<cylinder radius="0.05" length="0.2"/>-->
       </geometry>
@@ -117,5 +117,5 @@
   <!-- Joint 3 - Link 2 to Link 3 , fictive link (translation)-->
   <joint name="Axis3" type="prismatic">
-    <limit lower="-0.18" upper="0" effort="0" velocity="1.1"/><!-- -180 .. 0 mm , 1100mm/s which is 1.1 m/s -->
+    <limit lower="-0.18" upper="0" effort="10" velocity="1.1"/><!-- -180 .. 0 mm , 1100mm/s which is 1.1 m/s -->
     <parent link="link_2"/>
     <child link="link_3"/>
@@ -127,9 +127,9 @@
   <link name="link_3">
     <inertial>
-      <mass value="0.2"/>
-      <origin xyz="290.0 0.0 280.0" rpy="0.0 0.0 0.0"/>
-      <inertia ixx="0.00" ixy="0.0" ixz="0.0"
-               iyy="0.00" iyz="0.0"
-               izz="0.00"
+      <mass value="0.05"/>
+      <origin xyz="0 0 0.1975" rpy="0.0 0.0 0.0"/>
+      <inertia ixx="0.0001" ixy="0.0" ixz="0.0"
+               iyy="0.0001" iyz="0.0"
+               izz="0.0001"
       />
     </inertial>
@@ -140,5 +140,5 @@
   <!-- Joint 4 - Link 3 to Link 4 (rotation)-->
   <joint name="Axis4" type="revolute">
-    <limit lower="-6.98" upper="6.98" effort="0" velocity="43.63"/> <!-- +- 400° which is +- 6.98 rad , 2500°/s which is 43.63 rad/s -->
+    <limit lower="-6.98" upper="6.98" effort="5" velocity="43.63"/> <!-- +- 400° which is +- 6.98 rad , 2500°/s which is 43.63 rad/s -->
     <parent link="link_3"/>
     <child link="link_4"/>
@@ -150,8 +150,8 @@
   <link name="link_4">
     <inertial>
-      <mass value="0.0"/>
-      <origin xyz="0.0 0.0 0.0" rpy="0.0 0.0 0.0"/>
-      <inertia ixx="0.00" ixy="0.0" ixz="0.0"
-               iyy="0.00" iyz="0.0"
+      <mass value="0.18"/>
+      <origin xyz="0.0 0.0 0.1975" rpy="0.0 0.0 0.0"/>
+      <inertia ixx="0.0023" ixy="0.0" ixz="0.0"
+               iyy="0.0023" iyz="0.0"
                izz="0.00"
       />
@@ -165,5 +165,5 @@
     <visual>
       <geometry>
-      <mesh scale = "0.001 0.001 0.001" filename = "package://bme_ros_simple_arm/meshes/link3.dae"/>
+      <mesh scale = "1 1 1" filename = "package://bme_ros_simple_arm/meshes/Link3.dae"/>
         <!--<cylinder radius="0.025" length="0.25"/>-->
       </geometry>
@@ -195,5 +195,5 @@
     <visual>
       <geometry>
-        <mesh scale = "0.001 0.001 0.001" filename = "package://bme_ros_simple_arm/meshes/Gripper_body.dae"/>
+        <mesh scale = "1 1 1" filename = "package://bme_ros_simple_arm/meshes/M.dae"/>
         <!--<cylinder radius="0.025" length="0.25"/>-->
       </geometry>
@@ -204,5 +204,5 @@
 <!-- Left finger joint -->
   <joint name="left_finger_joint" type="prismatic">
-    <limit lower="0.006" upper="0" effort="100.0" velocity="4.0"/>
+    <limit lower="0.006" upper="0" effort="5.0" velocity="4.0"/>
     <parent link="link_E"/>
     <child link="left_finger"/>
@@ -228,5 +228,5 @@
     <visual>
       <geometry>
-        <mesh scale = "0.001 0.001 0.001" filename = "package://bme_ros_simple_arm/meshes/megfogo_pofa_1.dae"/>
+        <mesh scale = "1 1 1" filename = "package://bme_ros_simple_arm/meshes/MP1.dae"/>
       </geometry>
       <material name="blue"/>
@@ -246,5 +246,5 @@
   <!-- Right finger joint -->
   <joint name="right_finger_joint" type="prismatic">
-    <limit lower="0" upper="0.006" effort="100.0" velocity="4.0"/>
+    <limit lower="0" upper="0.006" effort="5.0" velocity="4.0"/>
     <parent link="link_E"/>
     <child link="right_finger"/>
@@ -270,5 +270,5 @@
     <visual>
       <geometry>
-        <mesh scale = "0.001 0.001 0.001" filename = "package://bme_ros_simple_arm/meshes/megfogo_pofa_2.dae"/>
+        <mesh scale = "1 1 1" filename = "package://bme_ros_simple_arm/meshes/MP2.dae"/>
       </geometry>
       <material name="blue"/>
@@ -288,5 +288,5 @@
   <!-- Gripper camera -->
   <joint type="fixed" name="gripper_camera_joint">
-    <origin xyz="0.0 0.0 0.0" rpy="0 -1.5707 0"/>
+    <origin xyz="0.0 0.0 -0.1" rpy="0 1.5707 0"/>
     <child link="gripper_camera_link"/>
     <parent link="link_E"/>
@@ -322,5 +322,5 @@
   <!-- Table camera -->
   <joint type="fixed" name="table_camera_joint">
-    <origin xyz="1.0 0.4 0.2" rpy="0 0 3.6652"/>
+    <origin xyz="0.275 0.275 1.0" rpy="0 1.5707 0"/>
     <child link="table_camera_link"/>
     <parent link="world"/>
