Commit message: Project rename

File: bme_ros_pp_project/urdf/mogi_arm.xacro (robot description, xacro)
@@ -2,5 +2,5 @@
 <robot name="mogi_arm" xmlns:xacro="http://www.ros.org/wiki/xacro">
   <!-- RViz colors -->
-  <xacro:include filename="$(find bme_ros_simple_arm)/urdf/materials.xacro" />
+  <xacro:include filename="$(find bme_ros_pp_project)/urdf/materials.xacro" />
   <!-- Global reference link -->
   <link name="world"/>
@@ -28,5 +28,5 @@
       <geometry>
         <!--<cylinder radius="0.15" length="0.05"/>-->
-        <mesh filename = "package://bme_ros_simple_arm/meshes/link0.dae"/>
+        <mesh filename = "package://bme_ros_pp_project/meshes/link0.dae"/>
       </geometry>
       <material name="grey"/>

File: bme_ros_pp_project/urdf/tomi_arm.xacro (robot description, xacro)
@@ -2,9 +2,9 @@
 <robot name="tomi_arm" xmlns:xacro="http://www.ros.org/wiki/xacro">
   <!-- RViz colors -->
-  <xacro:include filename="$(find bme_ros_simple_arm)/urdf/materials.xacro" />
+  <xacro:include filename="$(find bme_ros_pp_project)/urdf/materials.xacro" />
   <!-- Transmisions -->
-  <xacro:include filename="$(find bme_ros_simple_arm)/urdf/transmission.xacro" />
+  <xacro:include filename="$(find bme_ros_pp_project)/urdf/transmission.xacro" />
   <!-- Gazebo plugin -->
-  <xacro:include filename="$(find bme_ros_simple_arm)/urdf/tomi_arm.gazebo" />
+  <xacro:include filename="$(find bme_ros_pp_project)/urdf/tomi_arm.gazebo" />
   <!-- Global reference link -->
   <link name="world"/>
@@ -31,5 +31,5 @@
     <visual>
       <geometry>
-        <mesh scale = "1 1 1" filename = "package://bme_ros_simple_arm/meshes/Link0.dae"/>
+        <mesh scale = "1 1 1" filename = "package://bme_ros_pp_project/meshes/Link0.dae"/>
       </geometry>
       <material name="grey"/>
@@ -68,5 +68,5 @@
     <visual>
       <geometry>
-        <mesh scale = "1 1 1" filename = "package://bme_ros_simple_arm/meshes/Link1.dae"/>
+        <mesh scale = "1 1 1" filename = "package://bme_ros_pp_project/meshes/Link1.dae"/>
       </geometry>
       <material name="orange"/>
@@ -105,5 +105,5 @@
     <visual>
       <geometry>
-        <mesh scale = "1 1 1" filename = "package://bme_ros_simple_arm/meshes/Link2.dae"/>
+        <mesh scale = "1 1 1" filename = "package://bme_ros_pp_project/meshes/Link2.dae"/>
         <!--<cylinder radius="0.05" length="0.2"/>-->
       </geometry>
@@ -165,5 +165,5 @@
     <visual>
       <geometry>
-      <mesh scale = "1 1 1" filename = "package://bme_ros_simple_arm/meshes/Link3.dae"/>
+      <mesh scale = "1 1 1" filename = "package://bme_ros_pp_project/meshes/Link3.dae"/>
         <!--<cylinder radius="0.025" length="0.25"/>-->
       </geometry>
@@ -195,5 +195,5 @@
     <visual>
       <geometry>
-        <mesh scale = "1 1 1" filename = "package://bme_ros_simple_arm/meshes/M.dae"/>
+        <mesh scale = "1 1 1" filename = "package://bme_ros_pp_project/meshes/M.dae"/>
         <!--<cylinder radius="0.025" length="0.25"/>-->
       </geometry>
@@ -228,5 +228,5 @@
     <visual>
       <geometry>
-        <mesh scale = "1 1 1" filename = "package://bme_ros_simple_arm/meshes/MP1.dae"/>
+        <mesh scale = "1 1 1" filename = "package://bme_ros_pp_project/meshes/MP1.dae"/>
       </geometry>
       <material name="blue"/>
@@ -270,5 +270,5 @@
     <visual>
       <geometry>
-        <mesh scale = "1 1 1" filename = "package://bme_ros_simple_arm/meshes/MP2.dae"/>
+        <mesh scale = "1 1 1" filename = "package://bme_ros_pp_project/meshes/MP2.dae"/>
       </geometry>
       <material name="blue"/>
