Commit message: IKIN xyz OK, world correction

File: bme_ros_pp_project/urdf/tomi_arm.xacro (robot description, xacro)
@@ -222,7 +222,7 @@
     <collision>
       <geometry>
-        <box size=".04 .01 .08"/>
-      </geometry>
-      <origin xyz="0.0 0.0 0.0" rpy="0.0 0.0 0.0"/>
+        <box size="0.03 0.008 0.045"/>
+      </geometry>
+      <origin xyz="0.0 -0.02399 -0.12665" rpy="0.0 0.0 0.0"/>
     </collision>
     <visual>
@@ -264,7 +264,7 @@
     <collision>
       <geometry>
-        <box size=".04 .01 .08"/>
-      </geometry>
-      <origin xyz="0.0 0.0 0.0" rpy="0.0 0.0 0.0"/>
+        <box size="0.03 0.008 0.045"/>
+      </geometry>
+      <origin xyz="0.0 0.02399 -0.12665" rpy="0.0 0.0 0.0"/>
     </collision>
     <visual>

Commit message: img processing, gripper pub

File: bme_ros_pp_project/urdf/tomi_arm.xacro (robot description, xacro)
@@ -140,5 +140,5 @@
   <!-- Joint 4 - Link 3 to Link 4 (rotation)-->
   <joint name="Axis4" type="revolute">
-    <limit lower="-6.98" upper="6.98" effort="5" velocity="43.63"/> <!-- +- 400° which is +- 6.98 rad , 2500°/s which is 43.63 rad/s -->
+    <limit lower="-6.98" upper="6.98" effort="1" velocity="43.63"/> <!-- +- 400° which is +- 6.98 rad , 2500°/s which is 43.63 rad/s -->
     <parent link="link_3"/>
     <child link="link_4"/>
@@ -204,5 +204,5 @@
 <!-- Left finger joint -->
   <joint name="left_finger_joint" type="prismatic">
-    <limit lower="0.006" upper="0" effort="5.0" velocity="4.0"/>
+    <limit lower="0" upper="0.006" effort="100" velocity="4.0"/>
     <parent link="link_E"/>
     <child link="left_finger"/>
@@ -246,5 +246,5 @@
   <!-- Right finger joint -->
   <joint name="right_finger_joint" type="prismatic">
-    <limit lower="0" upper="0.006" effort="5.0" velocity="4.0"/>
+    <limit lower="0" upper="0.006" effort="100" velocity="4.0"/>
     <parent link="link_E"/>
     <child link="right_finger"/>

Commit message: pp works fine, but gripping is not the best

File: bme_ros_pp_project/urdf/tomi_arm.xacro (robot description, xacro)
@@ -204,8 +204,8 @@
 <!-- Left finger joint -->
   <joint name="left_finger_joint" type="prismatic">
-    <limit lower="0" upper="0.006" effort="100" velocity="4.0"/>
+    <limit lower="-0.016" upper="0.01" effort="100" velocity="4.0"/>
     <parent link="link_E"/>
     <child link="left_finger"/>
-    <axis xyz="0 1 0"/>
+    <axis xyz="0 -1 0"/>
     <origin xyz="0.0 0.00 0.00" />
   </joint>
@@ -246,8 +246,8 @@
   <!-- Right finger joint -->
   <joint name="right_finger_joint" type="prismatic">
-    <limit lower="0" upper="0.006" effort="100" velocity="4.0"/>
+    <limit lower="-0.0136" upper="0.01" effort="100" velocity="4.0"/>
     <parent link="link_E"/>
     <child link="right_finger"/>
-    <axis xyz="0 -1 0"/>
+    <axis xyz="0 1 0"/>
     <origin xyz="0.0 0.0 0.0" />
   </joint>

Commit message: write readme

File: bme_ros_pp_project/urdf/tomi_arm.xacro (robot description, xacro)
@@ -204,5 +204,5 @@
 <!-- Left finger joint -->
   <joint name="left_finger_joint" type="prismatic">
-    <limit lower="-0.016" upper="0.01" effort="100" velocity="4.0"/>
+    <limit lower="-0.016" upper="0.01" effort="400" velocity="4.0"/>
     <parent link="link_E"/>
     <child link="left_finger"/>
@@ -246,5 +246,5 @@
   <!-- Right finger joint -->
   <joint name="right_finger_joint" type="prismatic">
-    <limit lower="-0.0136" upper="0.01" effort="100" velocity="4.0"/>
+    <limit lower="-0.0136" upper="0.01" effort="400" velocity="4.0"/>
     <parent link="link_E"/>
     <child link="right_finger"/>
